File: pcb/motor.kicad_sch (KiCad schematic)
At the start: 9 parts, among them J1 Conn_01x04, J2 Conn_01x04, J3 Conn_01x04, J4 Conn_01x02, U4 Pico

Commit message: Change symbol name
Parts:
- U1, U2, U3: symbol motors:TMCSILENTSTEPSTICK -> motors:SILENTSTEPSTICK
Changed lines of the file:
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@@
     (stroke (width 0) (type default))
   )
-  (wire (pts (xy 208.28 73.66) (xy 201.93 73.66))
+  (wire (pts (xy 207.01 73.66) (xy 201.93 73.66))
     (stroke (width 0) (type default))
   )
@@
     (stroke (width 0) (type default))
   )
-  (wire (pts (xy 137.16 72.39) (xy 137.16 63.5))
+  (wire (pts (xy 135.89 72.39) (xy 135.89 63.5))
     (stroke (width 0) (type default))
   )
@@
     (stroke (width 0) (type default))
   )
-  (wire (pts (xy 137.16 72.39) (xy 128.27 72.39))
+  (wire (pts (xy 135.89 72.39) (xy 128.27 72.39))
     (stroke (width 0) (type default))
   )
@@
     (stroke (width 0) (type default))
   )
-  (wire (pts (xy 208.28 63.5) (xy 207.01 63.5))
-    (stroke (width 0) (type default))
-  )
-  (wire (pts (xy 137.16 63.5) (xy 135.89 63.5))
-    (stroke (width 0) (type default))
-  )
-  (wire (pts (xy 208.28 73.66) (xy 208.28 63.5))
+  (wire (pts (xy 207.01 73.66) (xy 207.01 63.5))
     (stroke (width 0) (type default))
   )
@@
     )
   )
-  (symbol (lib_id "motors:TMCSILENTSTEPSTICK") (at 55.88 48.26 0) (unit 1)
+  (symbol (lib_id "motors:SILENTSTEPSTICK") (at 54.61 48.26 0) (unit 1)
     (in_bom yes) (on_board yes) (dnp no) (fields_autoplaced)
     (property "Reference" "U1" (at 54.61 44.45 0)
       (effects (font (size 1.27 1.27)))
     )
-    (property "Value" "~" (at 53.34 48.26 0)
-      (effects (font (size 1.27 1.27)) hide)
-    )
-    (property "Footprint" "motors:SILENTSTEPSTICK" (at 53.34 48.26 0)
-      (effects (font (size 1.27 1.27)) hide)
-    )
-    (property "Datasheet" "" (at 53.34 48.26 0)
+    (property "Value" "~" (at 52.07 48.26 0)
+      (effects (font (size 1.27 1.27)) hide)
+    )
+    (property "Footprint" "motors:SILENTSTEPSTICK" (at 54.61 48.26 0)
+      (effects (font (size 1.27 1.27)) hide)
+    )
+    (property "Datasheet" "" (at 54.61 48.26 0)
       (effects (font (size 1.27 1.27)) hide)
     )
@@
     )
   )
-  (symbol (lib_id "motors:TMCSILENTSTEPSTICK") (at 196.85 46.99 0) (unit 1)
+  (symbol (lib_id "motors:SILENTSTEPSTICK") (at 195.58 46.99 0) (unit 1)
     (in_bom yes) (on_board yes) (dnp no) (fields_autoplaced)
     (property "Reference" "U3" (at 195.58 43.18 0)
       (effects (font (size 1.27 1.27)))
     )
-    (property "Value" "~" (at 194.31 46.99 0)
-      (effects (font (size 1.27 1.27)) hide)
-    )
-    (property "Footprint" "motors:SILENTSTEPSTICK" (at 194.31 46.99 0)
-      (effects (font (size 1.27 1.27)) hide)
-    )
-    (property "Datasheet" "" (at 194.31 46.99 0)
+    (property "Value" "~" (at 193.04 46.99 0)
+      (effects (font (size 1.27 1.27)) hide)
+    )
+    (property "Footprint" "motors:SILENTSTEPSTICK" (at 195.58 46.99 0)
+      (effects (font (size 1.27 1.27)) hide)
+    )
+    (property "Datasheet" "" (at 195.58 46.99 0)
       (effects (font (size 1.27 1.27)) hide)
     )
@@
     )
   )
-  (symbol (lib_id "motors:TMCSILENTSTEPSTICK") (at 125.73 46.99 0) (unit 1)
+  (symbol (lib_id "motors:SILENTSTEPSTICK") (at 124.46 46.99 0) (unit 1)
     (in_bom yes) (on_board yes) (dnp no) (fields_autoplaced)
     (property "Reference" "U2" (at 124.46 43.18 0)
       (effects (font (size 1.27 1.27)))
     )
-    (property "Value" "~" (at 123.19 46.99 0)
-      (effects (font (size 1.27 1.27)) hide)
-    )
-    (property "Footprint" "motors:SILENTSTEPSTICK" (at 123.19 46.99 0)
-      (effects (font (size 1.27 1.27)) hide)
-    )
-    (property "Datasheet" "" (at 123.19 46.99 0)
-      (effects (font (size 1.27 1.27)) hide)
-    )
+    (property "Value" "~" (at 121.92 46.99 0)
+      (effects (font (size 1.27 1.27)) hide)
+    )
+    (property "Footprint" "motors:SILENTSTEPSTICK" (at 124.46 46.99 0)
+      (effects (font (size 1.27 1.27)) hide)
+    )
+    (property "Datasheet" "" (at 124.46 46.99 0)
+      (effects (font (size 1.27 1.27)) hide)
+    )
